File: kicad/main/powerhammer_main.sch (KiCad schematic (older format))
At the start: 17 parts

Commit message: Updated schematic
Parts:
- removed K?: SOELENOID, symbol PINS_2
- removed Q?: MOSFET-SOT-23-3, SOT-23, symbol MOSFET-SOT-23-3
- removed R? (x2): 1k, symbol RESISTOR
- removed R?: 100k, symbol RESISTOR
- removed RV?: 10K, symbol POTENTIOMETER
- removed U?: ARDUINO_MICRO, symbol ARDUINO_MICRO
- added C1, C2: 8pF, symbol Device:C_Small
- added C3, C4: 1uF, symbol Device:C_Small
- added C5, C6, C7, C8, C9: 0.1uF, symbol Device:C_Small
- added J1: USB_B_Micro, symbol Connector:USB_B_Micro
- added K4: SOELENOID, symbol custom:PINS_2
- added Q1: MOSFET-SOT-23-3, SOT-23, symbol custom:MOSFET-SOT-23-3
- added R1, R2: 22, symbol custom:RSMALL
- added R3, R4: 10k, symbol custom:RSMALL
- added R5: 100k, symbol custom:RSMALL
- added R6, R7: 1k, symbol custom:RSMALL
- added RV1: POTENTIOMETER, symbol custom:POTENTIOMETER
- added SW1, SW2: SW_SPST, symbol Switch:SW_SPST
- added U1: ATmega32U4-AU, Package_QFP:TQFP-44_10x10mm_P0.8mm, symbol MCU_Microchip_ATmega:ATmega32U4-AU
- added X1: CRYSTAL_SMD_4PIN, symbol custom:CRYSTAL_SMD_4PIN
- DS1: renamed from DS?; symbol HD44780 -> custom:HD44780
- K1, K2, K3: renamed from K?; symbol PINS_3 -> custom:PINS_3
- K5, K6, K7, K8: renamed from K?; symbol PINS_2 -> custom:PINS_2
- SW3: renamed from SW?; symbol Rotary_Encoder -> powerhammer_main-rescue:Rotary_Encoder
- SW4: renamed from SW?; symbol Rotary_Encoder_Switch -> powerhammer_main-rescue:Rotary_Encoder_Switch
Connections:
- net labels added: +12V
- net labels removed: +24V, +8V
- wire segments 108 -> 164
- no-connect marks 7 -> 5

Commit message: Working on board layout
Parts:
- removed J1: USB_B_Micro, symbol Connector:USB_B_Micro
- removed SW1, SW2: SW_SPST, symbol Switch:SW_SPST
- added J1: USB_MINI_RIGHT, MF_Connectors:MF_Connectors-MINIUSB-RIGHT, symbol MF_Connectors:USB_MINI_RIGHT
- added SW1: RESET, MF_Switches:MF_Switches-TACT4.2MM, symbol MF_Switches:TACT_4.2MM
- added SW2: PROG, MF_Switches:MF_Switches-TACT4.2MM, symbol MF_Switches:TACT_4.2MM
- C1, C2, C3, C4, C5, C6, C7, C8, C9: footprint (none) -> MF_Passives:MF_Passives-C0603
- DS1: footprint (none) -> DigitalCave:HD44780
- K1, K2, K3, SW3: footprint (none) -> MF_Connectors:MF_Connectors-PTH_2.54MM_01X03
- K4: footprint (none) -> MF_Connectors:MF_Connectors-PTH_2.54MM_01X02
- K5: value BUTTON_1 -> BTN1; footprint (none) -> MF_Connectors:MF_Connectors-PTH_2.54MM_01X02
- K6: value BUTTON_2 -> BTN2; footprint (none) -> MF_Connectors:MF_Connectors-PTH_2.54MM_01X02
- K7: value BUTTON_3 -> BTN3; footprint (none) -> MF_Connectors:MF_Connectors-PTH_2.54MM_01X02
- K8: value BUTTON_4 -> BTN4; footprint (none) -> MF_Connectors:MF_Connectors-PTH_2.54MM_01X02
- Q1: footprint SOT-23 -> MF_Discrete_Semiconductor:MF_Discrete_Semiconductor-SOT-23-3
- R1, R2, R3, R4, R5, R6, R7: footprint (none) -> MF_Passives:MF_Passives-R0603
- RV1: footprint (none) -> MF_Passives:MF_Passives-TC33
- SW4: footprint (none) -> MF_Connectors:MF_Connectors-PTH_2.54MM_01X05
- U1: footprint Package_QFP:TQFP-44_10x10mm_P0.8mm -> MF_IC_Digital:MF_IC_Digital-TQFP44
- X1: footprint (none) -> MF_Frequency_Control:MF_Frequency_Control-5MMX3.2MM
Connections:
- wire segments 164 -> 176
- no-connect marks 5 -> 11

Commit message: sharing
Parts:
- added R? (x2): 1k, MF_Passives:MF_Passives-R0603, symbol custom:RSMALL
Connections:
- wire segments 176 -> 180
Changed lines of the file:
@@
 	8500 6450 7900 6450
-Wire Wire Line
-	7900 6450 7900 5550
-Wire Wire Line
-	7900 5550 3000 5550
 Wire Wire Line
 	6950 2650 6950 3950
@@
 Wire Wire Line
 	3400 5050 3500 5050
+$Comp
+L custom:RSMALL R?
+U 1 1 5BB6F1B4
+P 7900 5900
+F 0 "R?" H 7949 5939 40  0000 L CNN
+F 1 "1k" H 7949 5862 40  0000 L CNN
+F 2 "MF_Passives:MF_Passives-R0603" V 7830 5900 30  0001 C CNN
+F 3 "" H 7900 5950 30  0000 C CNN
+	1    7900 5900
+	-1   0    0    1
+$EndComp
+Wire Wire Line
+	7900 5550 7700 5550
+Wire Wire Line
+	7900 5800 7900 5550
+Wire Wire Line
+	7900 6000 7900 6450
+$Comp
+L custom:RSMALL R?
+U 1 1 5BB8922A
+P 7700 5900
+F 0 "R?" H 7749 5939 40  0000 L CNN
+F 1 "1k" H 7749 5862 40  0000 L CNN
+F 2 "MF_Passives:MF_Passives-R0603" V 7630 5900 30  0001 C CNN
+F 3 "" H 7700 5950 30  0000 C CNN
+	1    7700 5900
+	-1   0    0    1
+$EndComp
+Wire Wire Line
+	7700 5800 7700 5550
+$Comp
+L power:GND #PWR?
+U 1 1 5BB9AEEA
+P 7700 6150
+F 0 "#PWR?" H 7700 5900 50  0001 C CNN
+F 1 "GND" H 7700 6000 50  0000 C CNN
+F 2 "" H 7700 6150 50  0000 C CNN
+F 3 "" H 7700 6150 50  0000 C CNN
+	1    7700 6150
+	-1   0    0    -1
+$EndComp
+Wire Wire Line
+	7700 6000 7700 6150
+Connection ~ 7700 5550
+Wire Wire Line
+	7700 5550 3000 5550
 $EndSCHEMATC

Commit message: sharing
Parts:
- removed K5: BTN1, MF_Connectors:MF_Connectors-PTH_2.54MM_01X02, symbol custom:PINS_2
- removed K6: BTN2, MF_Connectors:MF_Connectors-PTH_2.54MM_01X02, symbol custom:PINS_2
- removed K7: BTN3, MF_Connectors:MF_Connectors-PTH_2.54MM_01X02, symbol custom:PINS_2
- removed K8: BTN4, MF_Connectors:MF_Connectors-PTH_2.54MM_01X02, symbol custom:PINS_2
- removed Q1: MOSFET-SOT-23-3, MF_Discrete_Semiconductor:MF_Discrete_Semiconductor-SOT-23-3, symbol custom:MOSFET-SOT-23-3
- removed SW4: UI_ENCODER, MF_Connectors:MF_Connectors-PTH_2.54MM_01X05, symbol powerhammer_main-rescue:Rotary_Encoder_Switch
- added J?: UI_ENCODER, MF_Connectors_PTH_2.54MM_01X06, symbol MF_Connectors:CON_01X06_PTH_2.54MM
- added Q?: MOSFET-SOT-23-3, MF_Discrete_Semiconductor:MF_Discrete_Semiconductor-SOT-23-3, symbol custom:MOSFET-SOT-23-3
- added R? (x2): 1k, MF_Passives:MF_Passives-R0603, symbol custom:RSMALL
- added R?: 200, MF_Passives:MF_Passives-R0603, symbol custom:RSMALL
Connections:
- net labels added: +24V, 24V_SENSE, CYL_ENCODER_A, CYL_ENCODER_B, DISP_D0, DISP_D1, DISP_D2, DISP_D3, DISP_D4, DISP_D5, DISP_D6, DISP_D7, DISP_EN, DISP_RS, PROG, SERVO_OUT, SOLENOID_EN, TDC_SENSOR, UI_ENCODER_A, UI_ENCODER_B, UI_ENCODER_BUTTON
- net labels removed: +12V
- wire segments 180 -> 188
- no-connect marks 11 -> 2
Other:
- moved on the sheet: U1

Commit message: sharing
Parts:
- added D?: DIODES_SOD-123, MF_Discrete_Semiconductor_SOD-123, symbol MF_Discrete_Semiconductor:DIODES_SOD-123
Connections:
- wire segments 188 -> 194
Changed lines of the file:
@@
 	3750 5850 8700 5850
 Wire Wire Line
-	9400 5400 9400 5600
+	9400 5400 9400 5500
 $Comp
 L power:+24V #PWR?
@@
 	8000 4950 8150 4950
 Wire Wire Line
-	8850 4950 8850 5300
-Wire Wire Line
-	8850 5300 9500 5300
-Wire Wire Line
 	8150 5250 8150 5350
 Wire Wire Line
 	8150 5050 8150 4950
 Connection ~ 8150 4950
-Wire Wire Line
-	8150 4950 8850 4950
 $Comp
 L power:GND #PWR?
@@
 Text Label 3850 3350 0    50   ~ 0
 CYL_ENCODER_B
+$Comp
+L MF_Discrete_Semiconductor:DIODES_SOD-123 D?
+U 1 1 5BB9DB13
+P 9100 5350
+F 0 "D?" V 9142 5262 45  0000 R CNN
+F 1 "DIODES_SOD-123" V 9058 5262 45  0000 R CNN
+F 2 "MF_Discrete_Semiconductor_SOD-123" H 9288 5429 20  0001 C CNN
+F 3 "" H 9100 5350 60  0001 C CNN
+	1    9100 5350
+	0    -1   -1   0
+$EndComp
+Wire Wire Line
+	9100 4950 9100 5200
+Wire Wire Line
+	9100 5200 9400 5200
+Wire Wire Line
+	9400 5200 9400 5300
+Wire Wire Line
+	9400 5300 9500 5300
+Wire Wire Line
+	8150 4950 9100 4950
+Wire Wire Line
+	9100 5500 9400 5500
+Connection ~ 9400 5500
+Wire Wire Line
+	9400 5500 9400 5600
+Wire Wire Line
+	9100 5500 9100 5450
+Wire Wire Line
+	9100 5250 9100 5200
+Connection ~ 9100 5200
 $EndSCHEMATC
